Commit message: Debugged gazebo pkg

File: solo_description/urdf/solo12.transmission.xacro (robot description, xacro)
@@ -5,5 +5,5 @@
     <transmission name="${prefix}_trans">
       <type>transmission_interface/SimpleTransmission</type>
-      <joint name="${prefix}_joint">
+      <joint name="${prefix}">
         <hardwareInterface>hardware_interface/EffortJointInterface</hardwareInterface>
       </joint>
